Commit message: Finished object recognition for DDW exhibition

File: urdf/workcell.xacro (robot description, xacro)
@@ -21,5 +21,5 @@
         <visual>
             <geometry>
-                <box size=".5 1.5 .5"/>
+                <box size=".5 1.1 .5"/>
             </geometry>
             <xacro:material_fanuc_white />
@@ -27,5 +27,5 @@
         <collision>
             <geometry>
-                <box size=".5 1.5 .5"/>
+                <box size=".5 1.1 .5"/>
             </geometry>
         </collision>
@@ -34,5 +34,5 @@
         <visual>
             <geometry>
-                <box size="1.5 .5 .5"/>
+                <box size=".93 .48 .53"/>
             </geometry>
             <xacro:material_fanuc_white />
@@ -40,12 +40,12 @@
         <collision>
             <geometry>
-                <box size="1.5 .5 .5"/>
+                <box size=".93 .48 .53"/>
             </geometry>
         </collision>
     </link>
-    <link name="ramp">
+    <link name="ramp_exit">
         <visual>
             <geometry>
-                <box size="1.5 .5 .01"/>
+                <box size=".92 .82 .115"/>
             </geometry>
             <xacro:material_fanuc_white />
@@ -53,5 +53,18 @@
         <collision>
             <geometry>
-                <box size="1.5 .5 .01"/>
+                <box size=".92 .82 .115"/>
+            </geometry>
+        </collision>
+    </link>
+    <link name="ramp_entrance">
+        <visual>
+            <geometry>
+                <box size=".5 1.70 .085"/>
+            </geometry>
+            <xacro:material_fanuc_white />
+        </visual>
+        <collision>
+            <geometry>
+                <box size=".5 1.70 .085"/>
             </geometry>
         </collision>
@@ -60,5 +73,5 @@
         <visual>
             <geometry>
-                <box size=".03 1.5 1.7"/>
+                <box size=".03 .03 1.7"/>
             </geometry>
             <xacro:material_fanuc_grey />
@@ -66,5 +79,5 @@
         <collision>
             <geometry>
-                <box size=".03 1.5 1.7"/>
+                <box size=".03 .03 1.7"/>
             </geometry>
         </collision>
@@ -73,5 +86,5 @@
         <visual>
             <geometry>
-                <box size=".012 1.5 .1"/>
+                <box size=".044 1.1 .14"/>
             </geometry>
             <xacro:material_fanuc_white />
@@ -79,5 +92,5 @@
         <collision>
             <geometry>
-                <box size=".012 1.5 .1"/>
+                <box size=".044 1.1 .14"/>
             </geometry>
         </collision>
@@ -86,5 +99,5 @@
         <visual>
             <geometry>
-                <box size=".012 1.5 .1"/>
+                <box size=".044 1.1 .14"/>
             </geometry>
             <xacro:material_fanuc_white />
@@ -92,5 +105,5 @@
         <collision>
             <geometry>
-                <box size=".012 1.5 .1"/>
+                <box size=".044 1.1 .14"/>
             </geometry>
         </collision>
@@ -112,17 +125,17 @@
     </link>
     <joint name="world_to_table" type="fixed">
-        <parent link="base_link"/>
+        <parent link="world"/>
         <child link="table"/>
-        <origin xyz="0.783 0.0 0.25" rpy="0 0 0"/>
+        <origin xyz="0.7665 0.02 0.25" rpy="0 0 0"/>
     </joint>
     <joint name="world_to_place" type="fixed">
-        <parent link="base_link"/>
+        <parent link="world"/>
         <child link="place_table"/>
-        <origin xyz="-.217 1.653 0.25" rpy="0 0 0"/>
+        <origin xyz="0 1.8 0.265" rpy="0 0 0"/>
     </joint>
     <joint name="ramp_table" type="fixed">
         <parent link="place_table"/>
-        <child link="ramp"/>
-        <origin xyz="0.0 -.4 0.35" rpy="-.6 0 0"/>
+        <child link="ramp_exit"/>
+        <origin xyz="0.0 -.67 0.405" rpy="-.227 0 0"/>
     </joint>
     <joint name="tripod_table" type="fixed">
@@ -131,13 +144,18 @@
         <origin xyz="0.45 0.0 0.6" rpy="0 0 0"/>
     </joint>
+    <joint name="entrance_ramp" type="fixed">
+        <parent link="table"/>
+        <child link="ramp_entrance"/>
+        <origin xyz="0.0 1.25 0.64" rpy=".43 0 0"/>
+    </joint>
     <joint name="bump1_table" type="fixed">
         <parent link="table"/>
         <child link="bumper1"/>
-        <origin xyz="0.256 0.0 0.25" rpy="0 0 0"/>
+        <origin xyz="0.272 0.0 0.25" rpy="0 0 0"/>
     </joint>
     <joint name="bump2_table" type="fixed">
         <parent link="table"/>
         <child link="bumper2"/>
-        <origin xyz="-0.256 0.0 0.25" rpy="0 0 0"/>
+        <origin xyz="-0.272 0.0 0.25" rpy="0 0 0"/>
     </joint>
     <joint name="ddw" type="fixed">
@@ -149,5 +167,5 @@
         <parent link="base_link"/>
         <child link="world"/>
-        <origin xyz="0.0 0.0 0.0" rpy="0 0 0"/>
+        <origin xyz="0.0 0.0 0.0" rpy="0 0 -.028"/>
     </joint>
     <joint name="eef_connect" type="fixed">
